Commit message: added camera to urdf

File: robot_bringup/urdf/robot.urdf.xacro (robot description, xacro)
@@ -8,7 +8,38 @@
     <!-- MAP -->
     <link name="map"/>
-    <!-- VELODYNE -->
+    <!-- CAMERA -->
+    <joint name="camera_joint" type="fixed">
+        <origin xyz="0 0.5 0.0" rpy="0 0 0" />
+        <parent link="map"/>
+        <child link="c270"/>
+    </joint>
+    <link name="c270">
+        <visual>
+            <origin xyz="0 0 0" rpy="0 0 0" />
+            <geometry>
+                <box size="0.015 0.05 0.02"/>
+            </geometry>
+            <material name="gray">
+                <color rgba="0.0 0.0 1.0 1.0" />
+            </material>
+        </visual>
+        <collision>
+            <origin xyz="0 0 0" rpy="0 0 0" />
+            <geometry>
+                <box size="0.015 0.05 0.02"/>
+            </geometry>
+        </collision>
+        <inertial>
+            <origin xyz="0 0 0" rpy="0 0 0" />
+            <mass value="1.0" />
+            <inertia
+                ixx="0.01" ixy="0.0" ixz="0.0"
+                iyy="0.02" iyz="0.0"
+                izz="0.03" />
+        </inertial>
+    </link>
+    <!-- LIDAR -->
     <joint name="velodyne_base_mount_joint" type="fixed">
-        <origin xyz="0 0 0.4" rpy="0 0 0" />
+        <origin xyz="0.5 0 0" rpy="0 0 0" />
         <parent link="map"/>
         <child link="velodyne_base_link"/>

Commit message: updated launch files

File: robot_bringup/urdf/robot.urdf.xacro (robot description, xacro)
@@ -1,4 +1,6 @@
 <?xml version="1.0"?>
 <robot xmlns:xacro="http://www.ros.org/wiki/xacro" name="robot">
+    <!-- INCLUDES -->
+    <xacro:include filename="$(find realsense2_description)/urdf/_d455.urdf.xacro" />
     <!-- ARGS -->
     <xacro:arg name="USE_WITH_SIM" default="false" />
@@ -9,34 +11,7 @@
     <link name="map"/>
     <!-- CAMERA -->
-    <joint name="camera_joint" type="fixed">
-        <origin xyz="0 0.5 0.0" rpy="0 0 0" />
-        <parent link="map"/>
-        <child link="c270"/>
-    </joint>
-    <link name="c270">
-        <visual>
-            <origin xyz="0 0 0" rpy="0 0 0" />
-            <geometry>
-                <box size="0.015 0.05 0.02"/>
-            </geometry>
-            <material name="gray">
-                <color rgba="0.0 0.0 1.0 1.0" />
-            </material>
-        </visual>
-        <collision>
-            <origin xyz="0 0 0" rpy="0 0 0" />
-            <geometry>
-                <box size="0.015 0.05 0.02"/>
-            </geometry>
-        </collision>
-        <inertial>
-            <origin xyz="0 0 0" rpy="0 0 0" />
-            <mass value="1.0" />
-            <inertia
-                ixx="0.01" ixy="0.0" ixz="0.0"
-                iyy="0.02" iyz="0.0"
-                izz="0.03" />
-        </inertial>
-    </link>
+    <xacro:sensor_d455 parent="map" use_nominal_extrinsics="$(arg use_nominal_extrinsics)" name="camera">
+      <origin xyz="0 0.5 0" rpy="0 0 y"/>
+    </xacro:sensor_d455>
     <!-- LIDAR -->
     <joint name="velodyne_base_mount_joint" type="fixed">

Commit message: updated urdf rviz launch etc

File: robot_bringup/urdf/robot.urdf.xacro (robot description, xacro)
@@ -11,6 +11,6 @@
     <link name="map"/>
     <!-- CAMERA -->
-    <xacro:sensor_d455 parent="map" use_nominal_extrinsics="$(arg use_nominal_extrinsics)" name="camera">
-      <origin xyz="0 0.5 0" rpy="0 0 y"/>
+    <xacro:sensor_d455 parent="map" use_nominal_extrinsics="True" name="camera">
+      <origin xyz="0 0.5 0" rpy="0 0 0"/>
     </xacro:sensor_d455>
     <!-- LIDAR -->

Commit message: Added Realsense D455 Support (#7)
* added realsense dependencies

* updated docker file with realsense dependencies

* updated launch files

* updated urdf rviz launch etc

* updated readme

* updated rosbag yaml for realsense messages

File: robot_bringup/urdf/robot.urdf.xacro (robot description, xacro)
@@ -1,4 +1,6 @@
 <?xml version="1.0"?>
 <robot xmlns:xacro="http://www.ros.org/wiki/xacro" name="robot">
+    <!-- INCLUDES -->
+    <xacro:include filename="$(find realsense2_description)/urdf/_d455.urdf.xacro" />
     <!-- ARGS -->
     <xacro:arg name="USE_WITH_SIM" default="false" />
@@ -9,34 +11,7 @@
     <link name="map"/>
     <!-- CAMERA -->
-    <joint name="camera_joint" type="fixed">
-        <origin xyz="0 0.5 0.0" rpy="0 0 0" />
-        <parent link="map"/>
-        <child link="c270"/>
-    </joint>
-    <link name="c270">
-        <visual>
-            <origin xyz="0 0 0" rpy="0 0 0" />
-            <geometry>
-                <box size="0.015 0.05 0.02"/>
-            </geometry>
-            <material name="gray">
-                <color rgba="0.0 0.0 1.0 1.0" />
-            </material>
-        </visual>
-        <collision>
-            <origin xyz="0 0 0" rpy="0 0 0" />
-            <geometry>
-                <box size="0.015 0.05 0.02"/>
-            </geometry>
-        </collision>
-        <inertial>
-            <origin xyz="0 0 0" rpy="0 0 0" />
-            <mass value="1.0" />
-            <inertia
-                ixx="0.01" ixy="0.0" ixz="0.0"
-                iyy="0.02" iyz="0.0"
-                izz="0.03" />
-        </inertial>
-    </link>
+    <xacro:sensor_d455 parent="map" use_nominal_extrinsics="True" name="camera">
+      <origin xyz="0 0.5 0" rpy="0 0 0"/>
+    </xacro:sensor_d455>
     <!-- LIDAR -->
     <joint name="velodyne_base_mount_joint" type="fixed">
