Commit message: updated naming structure

File: lidar_camera_calibration/urdf/robot.urdf.xacro (robot description, xacro)
@@ -28,10 +28,10 @@
       <visual>
         <geometry>
-          <mesh filename="file://$(find robot_bringup)/meshes/VLP16/VLP16_base_1.dae"/>
+          <mesh filename="file://$(find lidar_camera_calibration)/meshes/VLP16/VLP16_base_1.dae"/>
         </geometry>
       </visual>
       <visual>
         <geometry>
-          <mesh filename="file://$(find robot_bringup)/meshes/VLP16/VLP16_base_2.dae"/>
+          <mesh filename="file://$(find lidar_camera_calibration)/meshes/VLP16/VLP16_base_2.dae"/>
         </geometry>
       </visual>
@@ -57,5 +57,5 @@
         <origin xyz="0 0 -0.0377"/>
         <geometry>
-          <mesh filename="file://$(find robot_bringup)/meshes/VLP16/VLP16_scan.dae"/>
+          <mesh filename="file://$(find lidar_camera_calibration)/meshes/VLP16/VLP16_scan.dae"/>
         </geometry>
       </visual>

Commit message: added draft for calibration node

File: lidar_camera_calibration/urdf/robot.urdf.xacro (robot description, xacro)
@@ -10,8 +10,4 @@
     <!-- MAP -->
     <link name="map"/>
-    <!-- CAMERA -->
-    <xacro:sensor_d455 parent="map" use_nominal_extrinsics="True" name="camera">
-      <origin xyz="0 0.5 0" rpy="0 0 0"/>
-    </xacro:sensor_d455>
     <!-- LIDAR -->
     <joint name="velodyne_base_mount_joint" type="fixed">
@@ -61,3 +57,7 @@
       </visual>
     </link>
+    <!-- CAMERA -->
+    <xacro:sensor_d455 parent="velodyne" use_nominal_extrinsics="True" name="camera">
+      <origin xyz="0 0 0" rpy="0 0 0"/>
+    </xacro:sensor_d455>
 </robot>

Commit message: Added Calibration Package (#9)
* updated naming structure

* updated docker configs with dependencies

* merged sync sensors into main package

* added draft for calibration node

* updated claibraiton logic and added logging

* updated readme and added output file logic

File: lidar_camera_calibration/urdf/robot.urdf.xacro (robot description, xacro)
@@ -10,8 +10,4 @@
     <!-- MAP -->
     <link name="map"/>
-    <!-- CAMERA -->
-    <xacro:sensor_d455 parent="map" use_nominal_extrinsics="True" name="camera">
-      <origin xyz="0 0.5 0" rpy="0 0 0"/>
-    </xacro:sensor_d455>
     <!-- LIDAR -->
     <joint name="velodyne_base_mount_joint" type="fixed">
@@ -28,10 +24,10 @@
       <visual>
         <geometry>
-          <mesh filename="file://$(find robot_bringup)/meshes/VLP16/VLP16_base_1.dae"/>
+          <mesh filename="file://$(find lidar_camera_calibration)/meshes/VLP16/VLP16_base_1.dae"/>
         </geometry>
       </visual>
       <visual>
         <geometry>
-          <mesh filename="file://$(find robot_bringup)/meshes/VLP16/VLP16_base_2.dae"/>
+          <mesh filename="file://$(find lidar_camera_calibration)/meshes/VLP16/VLP16_base_2.dae"/>
         </geometry>
       </visual>
@@ -57,7 +53,11 @@
         <origin xyz="0 0 -0.0377"/>
         <geometry>
-          <mesh filename="file://$(find robot_bringup)/meshes/VLP16/VLP16_scan.dae"/>
+          <mesh filename="file://$(find lidar_camera_calibration)/meshes/VLP16/VLP16_scan.dae"/>
         </geometry>
       </visual>
     </link>
+    <!-- CAMERA -->
+    <xacro:sensor_d455 parent="velodyne_base_link" use_nominal_extrinsics="True" name="camera">
+      <origin xyz="0 0 0" rpy="0 0 0"/>
+    </xacro:sensor_d455>
 </robot>

Commit message: updated yaml and rviz configs

File: lidar_camera_calibration/urdf/robot.urdf.xacro (robot description, xacro)
@@ -7,12 +7,4 @@
     <!-- PROPERTIES -->
     <xacro:property name="PI" value="3.1415926535897931"/>
-    <!-- MAP -->
-    <link name="map"/>
-    <!-- LIDAR -->
-    <joint name="velodyne_base_mount_joint" type="fixed">
-        <origin xyz="0.5 0 0" rpy="0 0 0" />
-        <parent link="map"/>
-        <child link="velodyne_base_link"/>
-    </joint>
     <link name="velodyne_base_link">
       <inertial>

Commit message: added dummy map link

File: lidar_camera_calibration/urdf/robot.urdf.xacro (robot description, xacro)
@@ -7,4 +7,12 @@
     <!-- PROPERTIES -->
     <xacro:property name="PI" value="3.1415926535897931"/>
+    <!-- MAP -->
+    <link name="map"/>
+    <joint name="velodyne_joint" type="fixed">
+      <parent link="map"/>
+      <child link="velodyne_base_link"/>
+      <origin xyz="0 0 0" rpy="0 0 0"/>
+    </joint>
+    <!-- VELODYNE -->
     <link name="velodyne_base_link">
       <inertial>

Commit message: updated rviz setup

File: lidar_camera_calibration/urdf/robot.urdf.xacro (robot description, xacro)
@@ -58,5 +58,5 @@
     <!-- CAMERA -->
     <xacro:sensor_d455 parent="velodyne_base_link" use_nominal_extrinsics="True" name="camera">
-      <origin xyz="0 0 0" rpy="0 0 0"/>
+      <origin xyz="0.1 0.1 0.1" rpy="0 0 ${PI/3}"/>
     </xacro:sensor_d455>
 </robot>

Commit message: 2D-3D Correspondence Pipeline (#14)
* modified dependencies

* included headers for finding correspondences

* superglue python files

* superglue weights

* calc_tools cpp files

* preprocess and camera cpp files

* main cpp files for finding correspondences and rosbag preprocessing

* added ransac capabilities (#13)

* thirdparty to deprepos changes

* moved superglue models to dep_repos

* integrated pipeline sequence in Calibration launch file

* launch file modifies

* change in launch file again

* removed velodyne driver

* aesthetic changes

* more aesthetic changes

* updated readme

* added gpu passthrough to devcontianer

* updated yaml and rviz configs

* updated readme and media

* updated readme

* moved superglue frm root to home in dockerfile

* made rviz default to true

* mdoifed superglue path

* updated rviz setup

* added dummy map link

* updated rviz setup

---------

Co-authored-by: RoCon RRC <rocon.rrc@gmail.com>

File: lidar_camera_calibration/urdf/robot.urdf.xacro (robot description, xacro)
@@ -9,10 +9,10 @@
     <!-- MAP -->
     <link name="map"/>
-    <!-- LIDAR -->
-    <joint name="velodyne_base_mount_joint" type="fixed">
-        <origin xyz="0.5 0 0" rpy="0 0 0" />
-        <parent link="map"/>
-        <child link="velodyne_base_link"/>
+    <joint name="velodyne_joint" type="fixed">
+      <parent link="map"/>
+      <child link="velodyne_base_link"/>
+      <origin xyz="0 0 0" rpy="0 0 0"/>
     </joint>
+    <!-- VELODYNE -->
     <link name="velodyne_base_link">
       <inertial>
@@ -58,5 +58,5 @@
     <!-- CAMERA -->
     <xacro:sensor_d455 parent="velodyne_base_link" use_nominal_extrinsics="True" name="camera">
-      <origin xyz="0 0 0" rpy="0 0 0"/>
+      <origin xyz="0.1 0.1 0.1" rpy="0 0 ${PI/3}"/>
     </xacro:sensor_d455>
 </robot>
